File: KiCAD Circuits/ROBOT/BuckInverter.kicad_sch (KiCad schematic)
At the start: 4 parts

Commit message: circuitry update
Parts:
- C6: renamed from C?; footprint (none) -> Capacitor_THT:C_Axial_L5.1mm_D3.1mm_P15.00mm_Horizontal
- L1: renamed from L?; footprint (none) -> Inductor_THT:L_Axial_L11.0mm_D4.5mm_P15.24mm_Horizontal_Fastron_MECC
- gave numbers to parts that had none: 2
Changed lines of the file:
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@@
-(kicad_sch (version 20211123) (generator eeschema)
+(kicad_sch (version 20230121) (generator eeschema)
   (paper "A4")
   (junction (at 182.88 87.63) (diameter 0) (color 0 0 0 0)
@@
   )
   (wire (pts (xy 99.06 99.06) (xy 154.94 99.06))
-    (stroke (width 0) (type default) (color 0 0 0 0))
+    (stroke (width 0) (type default))
   )
   (wire (pts (xy 124.46 87.63) (xy 124.46 86.36))
-    (stroke (width 0) (type default) (color 0 0 0 0))
+    (stroke (width 0) (type default))
   )
   (wire (pts (xy 172.72 87.63) (xy 182.88 87.63))
-    (stroke (width 0) (type default) (color 0 0 0 0))
+    (stroke (width 0) (type default))
   )
   (wire (pts (xy 149.86 86.36) (xy 149.86 87.63))
-    (stroke (width 0) (type default) (color 0 0 0 0))
+    (stroke (width 0) (type default))
   )
   (wire (pts (xy 182.88 81.28) (xy 182.88 87.63))
-    (stroke (width 0) (type default) (color 0 0 0 0))
+    (stroke (width 0) (type default))
   )
   (wire (pts (xy 154.94 99.06) (xy 172.72 99.06))
-    (stroke (width 0) (type default) (color 0 0 0 0))
+    (stroke (width 0) (type default))
   )
   (wire (pts (xy 172.72 87.63) (xy 172.72 91.44))
-    (stroke (width 0) (type default) (color 0 0 0 0))
+    (stroke (width 0) (type default))
   )
   (wire (pts (xy 99.06 91.44) (xy 99.06 99.06))
-    (stroke (width 0) (type default) (color 0 0 0 0))
+    (stroke (width 0) (type default))
   )
   (wire (pts (xy 149.86 87.63) (xy 154.94 87.63))
-    (stroke (width 0) (type default) (color 0 0 0 0))
+    (stroke (width 0) (type default))
   )
   (wire (pts (xy 168.91 87.63) (xy 172.72 87.63))
-    (stroke (width 0) (type default) (color 0 0 0 0))
+    (stroke (width 0) (type default))
   )
   (wire (pts (xy 172.72 99.06) (xy 196.85 99.06))
-    (stroke (width 0) (type default) (color 0 0 0 0))
+    (stroke (width 0) (type default))
   )
   (wire (pts (xy 99.06 87.63) (xy 99.06 91.44))
-    (stroke (width 0) (type default) (color 0 0 0 0))
+    (stroke (width 0) (type default))
   )
   (wire (pts (xy 182.88 87.63) (xy 196.85 87.63))
-    (stroke (width 0) (type default) (color 0 0 0 0))
+    (stroke (width 0) (type default))
   )
   (wire (pts (xy 97.79 81.28) (xy 124.46 81.28))
-    (stroke (width 0) (type default) (color 0 0 0 0))
+    (stroke (width 0) (type default))
   )
   (wire (pts (xy 99.06 87.63) (xy 124.46 87.63))
-    (stroke (width 0) (type default) (color 0 0 0 0))
+    (stroke (width 0) (type default))
   )
   (wire (pts (xy 154.94 95.25) (xy 154.94 99.06))
-    (stroke (width 0) (type default) (color 0 0 0 0))
+    (stroke (width 0) (type default))
   )
   (wire (pts (xy 149.86 81.28) (xy 182.88 81.28))
-    (stroke (width 0) (type default) (color 0 0 0 0))
+    (stroke (width 0) (type default))
   )
   (wire (pts (xy 96.52 87.63) (xy 99.06 87.63))
-    (stroke (width 0) (type default) (color 0 0 0 0))
+    (stroke (width 0) (type default))
   )
   (wire (pts (xy 137.16 91.44) (xy 99.06 91.44))
-    (stroke (width 0) (type default) (color 0 0 0 0))
+    (stroke (width 0) (type default))
   )
   (wire (pts (xy 154.94 87.63) (xy 156.21 87.63))
-    (stroke (width 0) (type default) (color 0 0 0 0))
+    (stroke (width 0) (type default))
   )
-  (hierarchical_label "OUT+" (shape input) (at 196.85 87.63 0)
+  (hierarchical_label "OUT+" (shape input) (at 196.85 87.63 0) (fields_autoplaced)
     (effects (font (size 1.27 1.27)) (justify left))
   )
-  (hierarchical_label "OUT-" (shape input) (at 196.85 99.06 0)
+  (hierarchical_label "OUT-" (shape input) (at 196.85 99.06 0) (fields_autoplaced)
     (effects (font (size 1.27 1.27)) (justify left))
   )
-  (hierarchical_label "IN+" (shape input) (at 97.79 81.28 180)
+  (hierarchical_label "IN+" (shape input) (at 97.79 81.28 180) (fields_autoplaced)
     (effects (font (size 1.27 1.27)) (justify right))
   )
-  (hierarchical_label "IN-" (shape input) (at 96.52 87.63 180)
+  (hierarchical_label "IN-" (shape input) (at 96.52 87.63 180) (fields_autoplaced)
     (effects (font (size 1.27 1.27)) (justify right))
   )
   (symbol (lib_id "pspice:INDUCTOR") (at 162.56 87.63 0) (unit 1)
-    (in_bom yes) (on_board yes) (fields_autoplaced)
-    (property "Reference" "L?" (id 0) (at 162.56 81.28 0))
-    (property "Value" "INDUCTOR" (id 1) (at 162.56 83.82 0))
-    (property "Footprint" "" (id 2) (at 162.56 87.63 0)
+    (in_bom yes) (on_board yes) (dnp no) (fields_autoplaced)
+    (property "Reference" "L1" (at 162.56 81.28 0)
+      (effects (font (size 1.27 1.27)))
+    )
+    (property "Value" "INDUCTOR" (at 162.56 83.82 0)
+      (effects (font (size 1.27 1.27)))
+    )
+    (property "Footprint" "Inductor_THT:L_Axial_L11.0mm_D4.5mm_P15.24mm_Horizontal_Fastron_MECC" (at 162.56 87.63 0)
       (effects (font (size 1.27 1.27)) hide)
     )
-    (property "Datasheet" "~" (id 3) (at 162.56 87.63 0)
+    (property "Datasheet" "~" (at 162.56 87.63 0)
       (effects (font (size 1.27 1.27)) hide)
     )
     (pin "1")
     (pin "2")
+    (instances
+      (project "ROBOT"
+        (path "/4c06c41c-9bca-4047-a966-bb339025bf70/00f566c1-d8ca-4f41-9b53-ceec4a3d1976"
+          (reference "L1") (unit 1)
+        )
+      )
+    )
   )
   (symbol (lib_id "Diode:1N5822") (at 154.94 91.44 270) (unit 1)
-    (in_bom yes) (on_board yes) (fields_autoplaced)
-    (property "Reference" "D?" (id 0) (at 157.48 89.8524 90)
+    (in_bom yes) (on_board yes) (dnp no) (fields_autoplaced)
+    (property "Reference" "D1" (at 157.48 89.8524 90)
       (effects (font (size 1.27 1.27)) (justify left))
     )
-    (property "Value" "1N5824" (id 1) (at 157.48 92.3924 90)
+    (property "Value" "1N5824" (at 157.48 92.3924 90)
       (effects (font (size 1.27 1.27)) (justify left))
     )
-    (property "Footprint" "Diode_THT:D_DO-201AD_P15.24mm_Horizontal" (id 2) (at 150.495 91.44 0)
+    (property "Footprint" "Diode_THT:D_DO-201AD_P15.24mm_Horizontal" (at 150.495 91.44 0)
       (effects (font (size 1.27 1.27)) hide)
     )
-    (property "Datasheet" "http://www.vishay.com/docs/88526/1n5820.pdf" (id 3) (at 154.94 91.44 0)
+    (property "Datasheet" "http://www.vishay.com/docs/88526/1n5820.pdf" (at 154.94 91.44 0)
       (effects (font (size 1.27 1.27)) hide)
     )
     (pin "1")
     (pin "2")
+    (instances
+      (project "ROBOT"
+        (path "/4c06c41c-9bca-4047-a966-bb339025bf70/00f566c1-d8ca-4f41-9b53-ceec4a3d1976"
+          (reference "D1") (unit 1)
+        )
+      )
+    )
   )
   (symbol (lib_id "Device:C") (at 172.72 95.25 0) (unit 1)
-    (in_bom yes) (on_board yes) (fields_autoplaced)
-    (property "Reference" "C?" (id 0) (at 176.53 93.9799 0)
+    (in_bom yes) (on_board yes) (dnp no) (fields_autoplaced)
+    (property "Reference" "C6" (at 176.53 93.9799 0)
       (effects (font (size 1.27 1.27)) (justify left))
     )
-    (property "Value" "C" (id 1) (at 176.53 96.5199 0)
+    (property "Value" "C" (at 176.53 96.5199 0)
       (effects (font (size 1.27 1.27)) (justify left))
     )
-    (property "Footprint" "" (id 2) (at 173.6852 99.06 0)
+    (property "Footprint" "Capacitor_THT:C_Axial_L5.1mm_D3.1mm_P15.00mm_Horizontal" (at 173.6852 99.06 0)
       (effects (font (size 1.27 1.27)) hide)
     )
-    (property "Datasheet" "~" (id 3) (at 172.72 95.25 0)
+    (property "Datasheet" "~" (at 172.72 95.25 0)
       (effects (font (size 1.27 1.27)) hide)
     )
     (pin "1")
     (pin "2")
+    (instances
+      (project "ROBOT"
+        (path "/4c06c41c-9bca-4047-a966-bb339025bf70/00f566c1-d8ca-4f41-9b53-ceec4a3d1976"
+          (reference "C6") (unit 1)
+        )
+      )
+    )
   )
   (symbol (lib_id "Regulator_Switching:LM2596S-ADJ") (at 137.16 83.82 0) (unit 1)
-    (in_bom yes) (on_board yes) (fields_autoplaced)
-    (property "Reference" "U?" (id 0) (at 137.16 73.66 0))
-    (property "Value" "LM2596S-ADJ" (id 1) (at 137.16 76.2 0))
-    (property "Footprint" "Package_TO_SOT_SMD:TO-263-5_TabPin3" (id 2) (at 138.43 90.17 0)
+    (in_bom yes) (on_board yes) (dnp no) (fields_autoplaced)
+    (property "Reference" "U5" (at 137.16 73.66 0)
+      (effects (font (size 1.27 1.27)))
+    )
+    (property "Value" "LM2596S-ADJ" (at 137.16 76.2 0)
+      (effects (font (size 1.27 1.27)))
+    )
+    (property "Footprint" "Package_TO_SOT_SMD:TO-263-5_TabPin3" (at 138.43 90.17 0)
       (effects (font (size 1.27 1.27) italic) (justify left) hide)
     )
-    (property "Datasheet" "http://www.ti.com/lit/ds/symlink/lm2596.pdf" (id 3) (at 137.16 83.82 0)
+    (property "Datasheet" "http://www.ti.com/lit/ds/symlink/lm2596.pdf" (at 137.16 83.82 0)
       (effects (font (size 1.27 1.27)) hide)
     )
@@
     (pin "4")
     (pin "5")
+    (instances
+      (project "ROBOT"
+        (path "/4c06c41c-9bca-4047-a966-bb339025bf70/00f566c1-d8ca-4f41-9b53-ceec4a3d1976"
+          (reference "U5") (unit 1)
+        )
+      )
+    )
   )
 )
