File: KiCAD Circuits/ROBOT/IRBEAM.kicad_sch (KiCad schematic)
At the start: 14 parts

Commit message: circuitry update
Parts:
- removed R?: R_Variable, symbol Device:R_Variable
- added RV3: R_Potentiometer, Potentiometer_THT:Potentiometer_Bourns_3386C_Horizontal, symbol Device:R_Potentiometer
- C1, C2: renamed from C?; footprint (none) -> Capacitor_THT:C_Axial_L5.1mm_D3.1mm_P15.00mm_Horizontal
- R1, R2, R4, R5, R6, R7, R8, R9: renamed from R?; footprint (none) -> Resistor_THT:R_Axial_DIN0204_L3.6mm_D1.6mm_P2.54mm_Vertical
- U1, U2: renamed from U?; footprint (none) -> Package_SO:SSO-8_6.7x9.8mm_P2.54mm_Clearance8mm
- gave numbers to parts that had none: 1
Connections:
- net Artificial ground: now also RV3.1
- net at Q1.2 (E), U1.3 (+): now also RV3.2
