File: KiCAD Circuits/ROBOT/LPcircuitry.kicad_sch (KiCad schematic)
At the start: 5 parts

Commit message: circuitry update
Parts:
- C3, C4, C5: renamed from C?; footprint (none) -> Capacitor_THT:C_Axial_L5.1mm_D3.1mm_P15.00mm_Horizontal
- gave numbers to parts that had none: 2
